Commit message: go2 collision settings are fixed

File: resources/robots/go2/urdf/go2.urdf (robot description, URDF)
Before this commit: robot go2_description, 29 links, 28 joints
Links:
- link base: geometry collision box size=0.3762 0.0935 0.154; visual mesh filename=../dae/base.dae

Commit message: training parameters are fixed

File: resources/robots/go2/urdf/go2.urdf (robot description, URDF)
Before this commit: robot go2_description, 29 links, 28 joints
Links:
- link FL_hip: geometry visual mesh filename=../dae/hip.dae
- link FR_hip: geometry visual mesh filename=../dae/hip.dae
- link RL_hip: geometry visual mesh filename=../dae/hip.dae
- link RR_hip: geometry visual mesh filename=../dae/hip.dae
